Commit message: Rebase from 'upstream'

File: panda_moveit_config/config/panda_arm.xacro (robot description, xacro)
@@ -26,5 +26,5 @@
       <joint name="panda_joint4" value="0" />
       <joint name="panda_joint5" value="0" />
-      <joint name="panda_joint6" value="0" />
+      <joint name="panda_joint6" value="1.571" />
       <joint name="panda_joint7" value="0.785" />
     </group_state>
